Commit message: relative coordinate arch

File: body.urdf (robot description, URDF)
Before this commit: robot robot, 2 links, 1 joints
Links:
- removed link Leg
- removed link Torso
- added link Link_0, mass 1; collision box size=1 1 1; visual box size=1 1 1
- added link Link_1, mass 1; collision box size=1 1 1; visual box size=1 1 1
- added link Link_2, mass 1; collision box size=1 1 1; visual box size=1 1 1
- added link Link_3, mass 1; collision box size=1 1 1; visual box size=1 1 1
- added link Link_4, mass 1; collision box size=1 1 1; visual box size=1 1 1
- added link Link_5, mass 1; collision box size=1 1 1; visual box size=1 1 1
- added link Link_6, mass 1; collision box size=1 1 1; visual box size=1 1 1
Joints:
- removed joint Torso_Leg
- added joint Link_0_Link_1: type revolute, parent Link_0, child Link_1, origin xyz=0 0 1.0 rpy=0 0 0, axis 0 1 0, limit lower=-3.14159 upper=3.14159 effort=0.0 velocity=0.0
- added joint Link_1_Link_2: type revolute, parent Link_1, child Link_2, origin xyz=0 0 1 rpy=0 0 0, axis 0 1 0, limit lower=-3.14159 upper=3.14159 effort=0.0 velocity=0.0
- added joint Link_2_Link_3: type revolute, parent Link_2, child Link_3, origin xyz=0 0.5 0.5 rpy=0 0 0, axis 0 1 0, limit lower=-3.14159 upper=3.14159 effort=0.0 velocity=0.0
- added joint Link_3_Link_4: type revolute, parent Link_3, child Link_4, origin xyz=0 1 0 rpy=0 0 0, axis 0 1 0, limit lower=-3.14159 upper=3.14159 effort=0.0 velocity=0.0
- added joint Link_4_Link_5: type revolute, parent Link_4, child Link_5, origin xyz=0 0.5 -0.5 rpy=0 0 0, axis 0 1 0, limit lower=-3.14159 upper=3.14159 effort=0.0 velocity=0.0
- added joint Link_5_Link_6: type revolute, parent Link_5, child Link_6, origin xyz=0 0 -1 rpy=0 0 0, axis 0 1 0, limit lower=-3.14159 upper=3.14159 effort=0.0 velocity=0.0

Commit message: finished joints

File: body.urdf (robot description, URDF)
Before this commit: robot robot, 7 links, 6 joints
Links:
- removed link Link_0
- removed link Link_1
- removed link Link_2
- removed link Link_3
- removed link Link_4
- removed link Link_5
- removed link Link_6
- added link BackLeg, mass 1; collision box size=1 1 1; visual box size=1 1 1
- added link FrontLeg, mass 1; collision box size=1 1 1; visual box size=1 1 1
- added link Torso, mass 1; collision box size=1 1 1; visual box size=1 1 1
Joints:
- removed joint Link_0_Link_1
- removed joint Link_1_Link_2
- removed joint Link_2_Link_3
- removed joint Link_3_Link_4
- removed joint Link_4_Link_5
- removed joint Link_5_Link_6
- added joint Torso_BackLeg: type revolute, parent Torso, child BackLeg, origin xyz=1 0 1 rpy=0 0 0, axis 0 1 0, limit lower=-3.14159 upper=3.14159 effort=0.0 velocity=0.0
- added joint Torso_FrontLeg: type revolute, parent Torso, child FrontLeg, origin xyz=2 0 1 rpy=0 0 0, axis 0 1 0, limit lower=-3.14159 upper=3.14159 effort=0.0 velocity=0.0
